Commit message: Add dependencies to docker file, rebuild model

File: DockerROS/SimulationFiles/src/robot_desc/robot/robot.urdf (robot description, URDF)
Before this commit: robot project_robot, 6 links, 5 joints
Links:
- link combinedshoulder: mass 0.0159914 -> 0.0366356
- link hooplink: mass 0.0174 -> 0.0174423
