Commit message: Adjusted frames for the urdf file for calculations

File: DockerROS/SimulationFiles/install/robot_desc/share/robot_desc/robot/robot.urdf (robot description, URDF)
Before this commit: robot project_robot, 6 links, 5 joints
Joints:
- joint EEframe_frame: origin xyz=0.3 -0.0002 0.003 rpy=0 -0 2.97496e-65 -> xyz=0.3 -0.0002 0.003 rpy=3.42114e-49 -0 2.47619e-65
- joint elbow: limit lower=-2.30383 upper=2.30383 effort=10 velocity=10 -> lower=-2.29391 upper=2.31376 effort=10 velocity=10; origin xyz=0.0358 0.0085 0.0055 rpy=-1.71531e-32 1.36846e-48 2.42861e-17 -> xyz=0.298 -7.17848e-17 0.0025 rpy=-1.93211e-32 -1.45615e-32 -0.00992709
- joint elbowmotor: origin xyz=0.2622 0.0085 0 rpy=-3.14159 -0 -2.97496e-65 -> xyz=0 0 0.003 rpy=-2.73691e-48 -0 4.22857e-64
- joint shoulder: limit lower=-1.58072 upper=1.56087 effort=10 velocity=10 -> lower=-1.5708 upper=1.5708 effort=10 velocity=10; origin xyz=-0.0358 -0.0085 0.00548 rpy=-3.14159 1.2326e-32 3.13167 -> xyz=-2.16027e-17 4.996e-16 -0.00535 rpy=1.71531e-32 2.46519e-32 1.5708
- joint shouldermotor: origin xyz=0.0085 0.0678 0.09305 rpy=0 -0 -1.5708 -> xyz=0 0.1036 0.10388 rpy=0 -0 0

Commit message: sending files into ignition

File: DockerROS/SimulationFiles/install/robot_desc/share/robot_desc/robot/robot.urdf (robot description, URDF)
Before this commit: robot project_robot, 6 links, 5 joints
Links:
- link armbasemount: geometry collision mesh filename=file://home/Catcher/install/robot_desc/share/robot_desc/rob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; visual mesh filename=file://home/Catcher/install/robot_desc/share/robot_desc/rob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
- link combinedshoulder: mass 0.0159914 -> 0.0366356; geometry collision mesh filename=file://home/Catcher/install/robot_desc/share/robot_desc/rob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; visual mesh filename=file://home/Catcher/install/robot_desc/share/robot_desc/rob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
- link dynamixelmotor_withhorn: geometry collision mesh filename=file://home/Catcher/install/robot_desc/share/robot_desc/rob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; visual mesh filename=file://home/Catcher/install/robot_desc/share/robot_desc/rob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
- link dynamixelmotor_withhorn_2: geometry collision mesh filename=file://home/Catcher/install/robot_desc/share/robot_desc/rob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; visual mesh filename=file://home/Catcher/install/robot_desc/share/robot_desc/rob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
- link hooplink: mass 0.0174 -> 0.0174423; geometry collision mesh filename=file://home/Catcher/install/robot_desc/share/robot_desc/rob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; visual mesh filename=file://home/Catcher/install/robot_desc/share/robot_desc/rob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

File: DockerROS/SimulationFiles/src/robot_desc/robot/robot.urdf (robot description, URDF)
Before this commit: robot project_robot, 6 links, 5 joints
Links:
- link armbasemount: geometry collision mesh filename=file://home/Catcher/install/robot_desc/share/robot_desc/rob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; visual mesh filename=file://home/Catcher/install/robot_desc/share/robot_desc/rob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
- link combinedshoulder: geometry collision mesh filename=file://home/Catcher/install/robot_desc/share/robot_desc/rob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; visual mesh filename=file://home/Catcher/install/robot_desc/share/robot_desc/rob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
- link dynamixelmotor_withhorn: geometry collision mesh filename=file://home/Catcher/install/robot_desc/share/robot_desc/rob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; visual mesh filename=file://home/Catcher/install/robot_desc/share/robot_desc/rob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
- link dynamixelmotor_withhorn_2: geometry collision mesh filename=file://home/Catcher/install/robot_desc/share/robot_desc/rob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; visual mesh filename=file://home/Catcher/install/robot_desc/share/robot_desc/rob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
- link hooplink: geometry collision mesh filename=file://home/Catcher/install/robot_desc/share/robot_desc/rob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; visual mesh filename=file://home/Catcher/install/robot_desc/share/robot_desc/rob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
