Commit message: edit filepaths for simulation

File: DockerROS/SimulationFiles/src/robot_desc/TrueRobot/robot.urdf (robot description, URDF)
Before this commit: robot project_robot, 6 links, 5 joints
Links:
- link armbasemount: geometry collision mesh filename=file://src/robot_desc/TrueRobot/assets/armbasemount.stl; visual mesh filename=file://src/robot_desc/TrueRobot/assets/armbasemount.stl
- link dynamixelmotor_withhorn: geometry collision mesh filename=file://src/robot_desc/TrueRobot/assets/dynamixelmotor_withh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; visual mesh filename=file://src/robot_desc/TrueRobot/assets/dynamixelmotor_withh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
- link dynamixelmotor_withhorn_2: geometry collision mesh filename=file://src/robot_desc/TrueRobot/assets/dynamixelmotor_withh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; visual mesh filename=file://src/robot_desc/TrueRobot/assets/dynamixelmotor_withh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
- link hooplink: geometry collision mesh filename=file://src/robot_desc/TrueRobot/assets/hooplink.stl; visual mesh filename=file://src/robot_desc/TrueRobot/assets/hooplink.stl
- link shoulderlink: geometry collision mesh filename=file://src/robot_desc/TrueRobot/assets/bottomshoulderlink.s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; collision mesh filename=file://src/robot_desc/TrueRobot/assets/combinedshoulder.stl

Commit message: Fix PID loop

File: DockerROS/SimulationFiles/src/robot_desc/TrueRobot/robot.urdf (robot description, URDF)
Before this commit: robot project_robot, 6 links, 5 joints
Links:
- link armbasemount: mass 0.0616 -> 0.208294; geometry collision mesh filename=package://robot_desc/TrueRobot/assets/armbasemount.stl; visual mesh filename=package://robot_desc/TrueRobot/assets/armbasemount.stl
- link dynamixelmotor_withhorn: geometry collision mesh filename=package://robot_desc/TrueRobot/assets/dynamixelmotor_withho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; visual mesh filename=package://robot_desc/TrueRobot/assets/dynamixelmotor_withho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
- link dynamixelmotor_withhorn_2: geometry collision mesh filename=package://robot_desc/TrueRobot/assets/dynamixelmotor_withho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; visual mesh filename=package://robot_desc/TrueRobot/assets/dynamixelmotor_withho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
- link hooplink: mass 0.0174423 -> 0.0593038; geometry collision mesh filename=package://robot_desc/TrueRobot/assets/hooplink.stl; visual mesh filename=package://robot_desc/TrueRobot/assets/hooplink.stl
- link shoulderlink: mass 0.035888 -> 0.121158; geometry collision mesh filename=package://robot_desc/TrueRobot/assets/bottomshoulderlink.stl; collision mesh filename=package://robot_desc/TrueRobot/assets/combinedshoulder.stl
Joints:
- joint EEframe_frame: origin xyz=0.3 -0.0002 0.003 rpy=0 -0 2.77556e-17 -> xyz=0.3 -0.0002 0.003 rpy=0 2.18953e-47 1.73472e-18
- joint elbow: limit lower=-4.06046 upper=0.547209 effort=10 velocity=10 -> lower=-2.31425 upper=2.29342 effort=10 velocity=10; origin xyz=0.298 -1.82296e-17 -0.0025 rpy=3.14159 -3.42481e-17 -1.75663 -> xyz=0.298 9.55833e-16 -0.0025 rpy=3.14159 -6.69473e-32 -0.0104131
- joint elbowmotor: axis 0 0 -1 -> 0 0 1; origin xyz=-9.48677e-19 0 -0.003 rpy=-1.22465e-16 -1.67107e-24 -1.5708 -> xyz=7.89299e-17 -1.38778e-16 -0.003 rpy=2.46255e-32 -1.81497e-32 -1.55128
- joint shoulder: axis 0 0 -1 -> 0 0 1; limit lower=-1.5708 upper=1.5708 effort=10 velocity=10 -> lower=-1.59031 upper=1.55128 effort=10 velocity=10
